File: NEW.kicad_sch (KiCad schematic)
At the start: 16 parts, among them J1 Screw_Terminal_01x16, J2 Screw_Terminal_01x16, J3 buck converter, J4 Infrared, J5 BMI, J6 light sensor, Q1 PN2222A, U1 LM1117T-5.0, U2 ESP32-CAM

Commit message: Update KiCad project files
Parts:
- added C2, C3: C_Polarized_Small, Capacitor_THT:C_Disc_D3.8mm_W2.6mm_P2.50mm, symbol Device:C_Polarized_Small
- added J7: servo, Connector_PinHeader_2.54mm:PinHeader_1x03_P2.54mm_Vertical, symbol Connector:Screw_Terminal_01x03
- added J8: Screw_Terminal_01x03, Connector_PinHeader_2.54mm:PinHeader_1x03_P2.54mm_Vertical, symbol Connector:Screw_Terminal_01x03
- added J9: battery +, Connector_PinHeader_2.54mm:PinHeader_1x01_P2.54mm_Vertical, symbol Connector:Screw_Terminal_01x01
- J1, J2: footprint Connector_PinHeader_2.54mm:PinHeader_1x17_P2.54mm_Vertical -> Connector_PinHeader_2.54mm:PinHeader_1x16_P2.54mm_Vertical
- J4: footprint Connector_PinHeader_2.54mm:PinHeader_1x02_P2.54mm_Vertical -> Connector_PinHeader_2.54mm:PinHeader_1x03_P2.54mm_Vertical
Connections:
- net GND: now also Q1.3 (C), C2.2, C3.2, J7.3 (Pin_3), J8.3 (Pin_3)
- net VCC: now also C2.1, C3.1, J7.2 (Pin_2); no longer J4.2 (Pin_2)
- net at R1.2: now also U2.IO13; no longer U2.IO12
- net at J1.14 (Pin_14): now also J7.1 (Pin_1)
- net at J1.16 (Pin_16): now also J4.2 (Pin_2), J9.1 (Pin_1)
- net at J1.8 (Pin_8): now also J8.2 (Pin_2)
- net at J1.9 (Pin_9): now also J8.1 (Pin_1)
- no-connect marks 39 -> 35
